File: SplitSecondGame.kicad_pcb (KiCad board)
At the start: 2 copper layers, 50 x 100 mm, 77 parts, among them J1 BATTERY, J2 AVR-ISP-6, SW1 START, SW2 SELECT, SW3 UP, SW4 LEFT, SW5 RIGHT, SW6 DOWN, SW7 POWER, U1 ATmega328PB-AU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

Commit message: Routing, plot
Routing:
- net /R6: track 74.3 -> 67.4 mm
- net /R7: track 63.7 -> 68.5 mm
- net /R5: track 78.6 -> 74.6 mm
- net /O4: track 73.6 -> 76.6 mm, vias 0 -> 1
- net GND: track 182.0 -> 179.4 mm, vias 5 -> 2
- net /O2: track 61.5 -> 59.3 mm
- net /O3: track 44.8 -> 43.4 mm
- net /R2: track 74.1 -> 75.5 mm
- net VCC: track 102.5 -> 103.9 mm
- net /R3: track 67.4 -> 68.7 mm
- net /O0: track 67.1 -> 65.8 mm
- net SCK: track 75.9 -> 76.9 mm
- net /O5: track 56.4 -> 57.2 mm
- net /R10: track 87.6 -> 86.8 mm
- net /O1: track 53.9 -> 53.2 mm
Other:
- board text added: "LED Matrix Game Rev A 2019 Dominic Thibodeau dev@hotkeysoft.net"
